File: hardware/sb_ch340g/sb_ch340g.sch (KiCad schematic (older format))
At the start: 15 parts, among them P1 USB_OTG, P2 CONN_01X06, P3 CONN_01X13, P4 CONN_01X13, SW1 RESET_SW, U1 AMS1117-3.3, U2 CH340G, U3 RF200, Y1 12MHz

Commit message: Cleanup layout.
Parts:
- SW1: footprint (none) -> CrumpPrints:3x6x3.5mm_side_pushbutton_smd
- U3: footprint CrumpPrints:RF200_nosilk -> CrumpPrints:RF200
Changed lines of the file:
@@
 LIBS:valves
 LIBS:crumpschemes
+LIBS:sb_ch340g-cache
 EELAYER 25 0
 EELAYER END
@@
 F 0 "U3" H 4300 1700 60  0000 C CNN
 F 1 "RF200" H 4300 3200 60  0000 C CNN
-F 2 "CrumpPrints:RF200_nosilk" H 4250 2450 60  0001 C CNN
+F 2 "CrumpPrints:RF200" H 4250 2450 60  0001 C CNN
 F 3 "" H 4250 2450 60  0000 C CNN
 	1    4300 2450
@@
 F 0 "SW1" V 2300 3950 50  0000 C CNN
 F 1 "RESET_SW" V 2400 4050 50  0000 C CNN
-F 2 "" H 2350 4000 50  0001 C CNN
+F 2 "CrumpPrints:3x6x3.5mm_side_pushbutton_smd" H 2350 4000 50  0001 C CNN
 F 3 "" H 2350 4000 50  0000 C CNN
 	1    2350 3800
