File: hardware/snapcap.kicad_pcb (KiCad board)
At the start: 2 copper layers, 45.7 x 35.6 mm, 16 parts, among them P1 USB_OTG, P2 CONN_01X06, P3 CONN_01X13, P4 CONN_01X13, U1 AMS1117-3.3, U2 CH340G, U3 RF200, Y1 12MHz

Commit message: Start adding silk.
Parts:
- added G***: LOGO, CrumpPrintSymbols:Symbol_OSHW-Logo_12.5mm_NoText_Silkscreen, B.Cu at (152.7, 96.5)
- added svg2mod: G***, CrumpPrintSymbols:tc_30mm, F.Cu at (154.9, 108.6)
- added svg2mod: G***, CrumpPrintSymbols:tc_30mm, B.Cu at (160.8, 114.7)
Other:
- board text added: "@"
- board text added: "CC-BY-SA 4.0"
- board text added: "TRY. LEARN. REPEAT."
- board text added: "snapcap"
- board text added: "tylercrumpton"
- board text added: "v1.0"
