File: hardware/slimjim2.kicad_pcb (KiCad board)
At the start: 2 copper layers, 45.7 x 35.6 mm, 19 parts, among them P1 USB_OTG, P2 CONN_01X06, P3 CONN_01X13, P4 CONN_01X13, U1 AMS1117-3.3, U2 CH340G, U3 RF200, Y1 12MHz

Commit message: Finish up silk.
Parts:
- removed the svg2mod at (160.8, 114.7)
- added G***: LOGO, CrumpPrintSymbols:tc_wide_18mm, B.Cu at (153.3, 89.9)
- moved G*** 8.75 mm to (148.6, 104.3)
- moved P4 1.27 mm to (167.6, 88.9)
- moved P3 1.27 mm to (129.5, 88.9)
Routing:
- net GPIO19: track 5.25 -> 3.98 mm
- net GPIO16: track 6.15 -> 4.88 mm
- net 3V3: track 22.1 -> 20.8 mm
- net SNAP_RST: track 50.9 -> 49.6 mm
- net GPIO18: track 5.70 -> 4.43 mm
- net GPIO17: track 5.92 -> 4.65 mm
- net GPIO5: track 6.15 -> 4.88 mm
- net GPIO0: track 5.03 -> 3.76 mm
- net GPIO2: track 5.48 -> 4.21 mm
- net GPIO3: track 5.70 -> 4.43 mm
- net GPIO4: track 5.92 -> 4.65 mm
- net GPIO1: track 5.25 -> 3.98 mm
- net 5V: track 52.6 -> 51.5 mm
- net GPIO12: track 7.79 -> 7.26 mm
- net GPIO15: track 6.37 -> 5.84 mm
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Other:
- board size 45.7 x 35.6 mm -> 48.3 x 35.6 mm
- board text added: "3V3"
- board text added: "5V"
- board text added: "IO0"
- board text added: "IO1"
- board text added: "IO10"
- board text added: "IO11"
- board text added: "IO12"
- board text added: "IO13"
- board text added: "IO14"
- board text added: "IO15"
- board text added: "IO16"
- board text added: "IO17"
- board text added: "IO18"
- board text added: "IO19"
- board text added: "IO2"
- board text added: "IO3"
- board text added: "IO4"
- board text added: "IO5"
- board text added: "IO6"
- board text added: "IO7"
- board text added: "IO8"
- board text added: "IO9"
- board text added: "RST"
- board text added: "slimjim2"
- board text added: "v2.0"
- board text removed: "snapcap"
- board text removed: "v1.0"
