File: hardware/slimjim2.sch (KiCad schematic (older format))
At the start: 15 parts, among them P1 USB_OTG, P2 CONN_01X06, P3 CONN_01X13, P4 CONN_01X13, SW1 RESET_SW, U1 AMS1117-3.3, U2 CH340G, U3 RF200, Y1 12MHz

Commit message: Update for KiCad5.
Parts:
- C1, C2, C3, C4, C5: symbol C_Small -> Device:C_Small
- P1: symbol USB_OTG -> slimjim2-rescue:USB_OTG
- P2: symbol CONN_01X06 -> slimjim2-rescue:CONN_01X06
- P3, P4: symbol CONN_01X13 -> slimjim2-rescue:CONN_01X13
- R1: symbol R_Small -> Device:R_Small
- SW1: symbol SW_PUSH_SMALL_H -> slimjim2-rescue:SW_PUSH_SMALL_H
- U1: symbol LM1117-3.3 -> slimjim2-rescue:LM1117-3.3
- U2: symbol CH340G -> crumpschemes:CH340G
- U3: symbol RF200 -> crumpschemes:RF200
- Y1: symbol 4-pin_Crystal_Oscillator -> crumpschemes:4-pin_Crystal_Oscillator
Changed lines of the file:
@@
-EESchema Schematic File Version 2
-LIBS:power
-LIBS:device
-LIBS:transistors
-LIBS:conn
-LIBS:linear
-LIBS:regul
-LIBS:74xx
-LIBS:cmos4000
-LIBS:adc-dac
-LIBS:memory
-LIBS:xilinx
-LIBS:microcontrollers
-LIBS:dsp
-LIBS:microchip
-LIBS:analog_switches
-LIBS:motorola
-LIBS:texas
-LIBS:intel
-LIBS:audio
-LIBS:interface
-LIBS:digital-audio
-LIBS:philips
-LIBS:display
-LIBS:cypress
-LIBS:siliconi
-LIBS:opto
-LIBS:atmel
-LIBS:contrib
-LIBS:valves
-LIBS:crumpschemes
+EESchema Schematic File Version 4
 LIBS:slimjim2-cache
-EELAYER 25 0
+EELAYER 29 0
 EELAYER END
 $Descr A4 11693 8268
@@
 $EndDescr
 $Comp
-L CH340G U2
+L crumpschemes:CH340G U2
 U 1 1 59C35380
 P 7100 2050
@@
 5V
 $Comp
-L GND #PWR01
+L power:GND #PWR01
 U 1 1 59C362D1
 P 6350 2550
@@
 $EndComp
 $Comp
-L LM1117-3.3 U1
+L slimjim2-rescue:LM1117-3.3 U1
 U 1 1 59C36518
 P 2200 1900
@@
 	6250 2900 6300 2900
 Wire Wire Line
-	1650 1900 1900 1900
+	1650 1900 1750 1900
 Text GLabel 2750 1900 2    60   Input ~ 0
 3V3
 Wire Wire Line
-	2500 1900 2750 1900
+	2500 1900 2600 1900
 Text GLabel 6150 1800 0    60   Input ~ 0
 3V3
 $Comp
-L GND #PWR02
+L power:GND #PWR02
 U 1 1 59C36883
 P 6450 1850
@@
 	6300 2000 6300 1800
 Wire Wire Line
-	6150 1800 6600 1800
+	6150 1800 6300 1800
 Connection ~ 6300 1800
 $Comp
-L GND #PWR03
+L power:GND #PWR03
 U 1 1 59C36A04
 P 2200 2300
@@
 $EndComp
 Wire Wire Line
-	2200 2200 2200 2300
-$Comp
-L C_Small C4
+	2200 2200 2200 2250
+$Comp
+L Device:C_Small C4
 U 1 1 59C36C51
 P 2000 5150
@@
 $EndComp
 $Comp
-L C_Small C5
+L Device:C_Small C5
 U 1 1 59C36EE2
 P 2400 5150
@@
 $EndComp
 $Comp
-L GND #PWR04
+L power:GND #PWR04
 U 1 1 59C37019
 P 2200 5350
@@
 $EndComp
 Wire Wire Line
-	2000 5300 2400 5300
+	2000 5300 2200 5300
 Wire Wire Line
 	2200 5300 2200 5350
@@
 CH340 USB-UART Converter
 $Comp
-L RF200 U3
+L crumpschemes:RF200 U3
 U 1 1 59C37A6F
 P 4300 2450
@@
 	4850 2000 4900 2000
 $Comp
-L GND #PWR05
+L power:GND #PWR05
 U 1 1 59C37D81
 P 5000 1800
@@
 	4900 1800 5000 1800
 $Comp
-L GND #PWR06
+L power:GND #PWR06
 U 1 1 59C37DD2
 P 3600 1800
@@
 	3900 4950 3950 4950
 $Comp
-L GND #PWR07
+L power:GND #PWR07
 U 1 1 59C38D61
 P 3800 4050
@@
 	4700 4250 4750 4250
 $Comp
-L GND #PWR08
+L power:GND #PWR08
 U 1 1 59C38DC8
 P 4850 4050
@@
 	7600 1800 7650 1800
 $Comp
-L C_Small C3
+L Device:C_Small C3
 U 1 1 59C39011
 P 2100 3500
@@
 SNAP_RST
 Wire Wire Line
-	2200 3500 2450 3500
+	2200 3500 2350 3500
 Text GLabel 7650 2200 2    60   Input ~ 0
 DTR
@@
 DTR
 $Comp
-L R_Small R1
+L Device:R_Small R1
 U 1 1 59C39813
 P 2350 3250
@@
 $EndComp
 Wire Wire Line
-	2350 3350 2350 3650
+	2350 3350 2350 3500
 Connection ~ 2350 3500
 $Comp
-L GND #PWR09
+L power:GND #PWR09
 U 1 1 59C39931
 P 2350 4000
@@
 Text Notes 1900 2900 0    60   ~ 0
 Reset Circuit
-$Comp
-L SW_PUSH_SMALL_H SW1
-U 1 1 59C39D4B
-P 2350 3800
-F 0 "SW1" V 2300 3950 50  0000 C CNN
-F 1 "RESET_SW" V 2400 4050 50  0000 C CNN
-F 2 "CrumpPrints:3x6x3.5mm_side_pushbutton_smd" H 2350 4000 50  0001 C CNN
-F 3 "" H 2350 4000 50  0000 C CNN
-	1    2350 3800
-	0    1    1    0
-$EndComp
 Wire Wire Line
 	2350 3950 2350 4000
@@
 	4750 5350 4700 5350
 $Comp
-L CONN_01X13 P3
+L slimjim2-rescue:CONN_01X13 P3
 U 1 1 59C3ADB8
 P 4150 4750
@@
 $EndComp
 $Comp
-L CONN_01X13 P4
+L slimjim2-rescue:CONN_01X13 P4
 U 1 1 59C3AE29
 P 4500 4750
@@
 	2350 3050 2300 3050
 $Comp
-L C_Small C1
+L Device:C_Small C1
 U 1 1 59C3BE38
 P 1750 2100
@@
 Connection ~ 1750 1900
 $Comp
-L C_Small C2
+L Device:C_Small C2
 U 1 1 59C3C5C1
 P 2600 2100
@@
 	1750 2200 1750 2250
 Wire Wire Line
-	1750 2250 2600 2250
-$Comp
-L CONN_01X06 P2
+	1750 2250 1850 2250
+$Comp
+L slimjim2-rescue:CONN_01X06 P2
 U 1 1 59C4AFE2
 P 6800 4250
@@
 NoConn ~ 5850 2300
 $Comp
-L PWR_FLAG #FLG010
+L power:PWR_FLAG #FLG010
 U 1 1 59C4C2B6
 P 1850 2300
@@
 Connection ~ 1850 2250
 $Comp
-L GND #PWR011
+L power:GND #PWR011
 U 1 1 59C4CB59
 P 6450 4000
@@
 Serial Breakout Header
 $Comp
-L USB_OTG P1
+L slimjim2-rescue:USB_OTG P1
 U 1 1 59C4F14C
 P 5950 2700
@@
 	1750 2000 1750 1900
 Wire Wire Line
-	2350 4850 2450 4850
-Wire Wire Line
-	1950 4850 2050 4850
-$Comp
-L 4-pin_Crystal_Oscillator Y1
+	2350 4850 2400 4850
+Wire Wire Line
+	1950 4850 2000 4850
+$Comp
+L crumpschemes:4-pin_Crystal_Oscillator Y1
 U 1 1 59C50040
 P 2200 4850
@@
 Wire Wire Line
 	2400 5300 2400 5250
+Wire Wire Line
+	6300 1800 6600 1800
+Wire Wire Line
+	2200 5300 2400 5300
+Wire Wire Line
+	2350 3500 2450 3500
+Wire Wire Line
+	2350 3500 2350 3650
+Wire Wire Line
+	1750 1900 1900 1900
+Wire Wire Line
+	2200 2250 2200 2300
+Wire Wire Line
+	2200 2250 2600 2250
+Wire Wire Line
+	2600 1900 2750 1900
+Wire Wire Line
+	1850 2250 2200 2250
+Wire Wire Line
+	2400 4850 2450 4850
+Wire Wire Line
+	2000 4850 2050 4850
+$Comp
+L slimjim2-rescue:SW_PUSH_SMALL_H SW1
+U 1 1 59C39D4B
+P 2350 3800
+F 0 "SW1" V 2300 3950 50  0000 C CNN
+F 1 "RESET_SW" V 2400 4050 50  0000 C CNN
+F 2 "CrumpPrints:3x6x3.5mm_side_pushbutton_smd" H 2350 4000 50  0001 C CNN
+F 3 "" H 2350 4000 50  0000 C CNN
+	1    2350 3800
+	0    1    1    0
+$EndComp
 $EndSCHEMATC
