File: hardware/_saved_slimjim2.sch (KiCad schematic (older format))
At the start: 18 parts, among them J1 USB_C_Receptacle_USB2.0, P2 CONN_01X06, P3 CONN_01X13, P4 CONN_01X13, SW1 RESET_SW, U1 AMS1117-3.3, U2 CH340G, U3 RF200, Y1 12MHz

Commit message: Update PCB with USB-C part.
Parts:
- J1: footprint (none) -> CrumpPrints:USB_C_Receptacle_SMD_THT
Changed lines of the file:
@@
 F 0 "J1" H 6550 3100 50  0000 C CNN
 F 1 "USB_C_Receptacle_USB2.0" H 6550 3000 50  0000 C CNN
-F 2 "" H 6700 2250 50  0001 C CNN
+F 2 "CrumpPrints:USB_C_Receptacle_SMD_THT" H 6700 2250 50  0001 C CNN
 F 3 "https://www.usb.org/sites/default/files/documents/usb_type-c.zip" H 6700 2250 50  0001 C CNN
 	1    6550 2250
